Commit message: Add initial bumperbot simulation and control configurations
- Updated CMakeLists.txt for bumperbot_description
- Modified bumperbot.urdf.xacro for improved URDF structure
- Added new bumperbot_controller package
- Added launch file for Gazebo simulation
- Added model files for bumperbot
- Added new URDF files for Gazebo and ROS2 control

File: bumperbot_description/urdf/bumperbot.urdf.xacro (robot description, xacro)
@@ -1,6 +1,13 @@
 <?xml version="1.0"?>
 <robot xmlns:xacro="http://www.ros.org/wiki/xacro" name="bumperbot">
+    <xacro:include filename="$(find bumperbot_description)/urdf/bumperbot_gazebo.xacro"/>
+    <xacro:include filename="$(find bumperbot_description)/urdf/bumperbot_ros2_control.xacro"/>
     <link name="base_footprint"/>
     <link name="base_link">
+        <inertial>
+            <origin xyz="0 0 0.04" rpy="0.0 0.25 0.3"/>
+            <mass value="8.2573504e-01"/>
+            <inertia ixx="2.2124416e-02" ixy="-1.2294101e-04" ixz="3.4938785e-04" iyy="2.1193702e-02" iyz="-5.0120904e-05" izz="2.0064271e-02"/>
+        </inertial>
         <visual>
             <origin xyz="0 0 0" rpy="0 0 0"/>
@@ -9,11 +16,22 @@
             </geometry>
         </visual>
+        <collision>
+            <origin xyz="0 0 0" rpy="0 0 0"/>
+            <geometry>
+                <mesh filename="file://$(find bumperbot_description)/meshes/base_link.STL"/>
+            </geometry>
+        </collision>
     </link>
     <joint name="base_joint" type="fixed">
         <parent link="base_footprint"/>
         <child link="base_link"/>
-        <origin xyz="0 0 0.33" rpy="0 0 0"/>
+        <origin xyz="0 0 0.033" rpy="0 0 0"/>
     </joint>
     <link name="wheel_right_link">
+        <inertial>
+            <origin xyz="0 -0.014 0" rpy="0 0 0"/>
+            <mass value="0.0530086090966721"/>
+            <inertia ixx="1.88176298336665E-05" ixy="-4.8444933029987E-10" ixz="1.88163708851143E-08" iyy="3.11510738647764E-05" iyz="-6.93560663069607E-11" izz="1.8801969558182E-05"/>
+        </inertial>
         <visual>
             <origin xyz="0 0 0" rpy="1.57 0 0"/>
@@ -22,4 +40,10 @@
             </geometry>
         </visual>
+        <collision>
+            <origin xyz="0 -0.015 0" rpy="1.57 0 0"/>
+            <geometry>
+                <sphere radius="0.033"/>
+            </geometry>
+        </collision>
     </link>
     <joint name="wheel_right_joint" type="continuous">
@@ -30,4 +54,9 @@
     </joint>
     <link name="wheel_left_link">
+        <inertial>
+            <origin xyz="0 0.014 0" rpy="0 0 0"/>
+            <mass value="0.0530086043217644"/>
+            <inertia ixx="1.8792911368909E-05" ixy="3.31256392204584E-10" ixz="-1.14082001662767E-08" iyy="3.11510738759073E-05" iyz="-3.60499245082192E-10" izz="1.88266886146847E-05"/>
+        </inertial>
         <visual>
             <origin xyz="0 0 0" rpy="-1.57 0 0"/>
@@ -36,4 +65,10 @@
             </geometry>
         </visual>
+        <collision>
+            <origin xyz="0 0.015 0" rpy="1.57 0 0"/>
+            <geometry>
+                <sphere radius="0.033"/>
+            </geometry>
+        </collision>
     </link>
     <joint name="wheel_left_joint" type="continuous">
@@ -44,4 +79,9 @@
     </joint>
     <link name="caster_front_link">
+        <inertial>
+            <origin xyz="3.89968128948481E-07 2.40073004698083E-07 0.00219173397061506" rpy="0 0 0"/>
+            <mass value="1.44379265037903E-06"/>
+            <inertia ixx="7.23075276010246E-11" ixy="-6.10956883467859E-16" ixz="2.22849693525031E-15" iyy="3.8713793085917E-11" iyz="2.93909858781952E-15" izz="1.00967486676306E-10"/>
+        </inertial>
         <visual>
             <origin xyz="0 0 0" rpy="0 0 0"/>
@@ -50,4 +90,10 @@
             </geometry>
         </visual>
+        <collision>
+            <origin xyz="0 0 0" rpy="0 0 0"/>
+            <geometry>
+                <sphere radius="0.005"/>
+            </geometry>
+        </collision>
     </link>
     <joint name="caster_front_joint" type="fixed">
@@ -57,4 +103,9 @@
     </joint>
     <link name="caster_rear_link">
+        <inertial>
+            <origin xyz="3.8996812895542E-07 2.40073004698083E-07 0.00219173397061509" rpy="0 0 0"/>
+            <mass value="1.44379265037902E-06"/>
+            <inertia ixx="7.23075276010246E-11" ixy="-6.10956872363424E-16" ixz="2.22849693527207E-15" iyy="3.87137930859167E-11" iyz="2.939098587861E-15" izz="1.00967486676306E-10"/>
+        </inertial>
         <visual>
             <origin xyz="0 0 0" rpy="0 0 0"/>
@@ -63,4 +114,10 @@
             </geometry>
         </visual>
+        <collision>
+            <origin xyz="0 0 0" rpy="0 0 0"/>
+            <geometry>
+                <sphere radius="0.005"/>
+            </geometry>
+        </collision>
     </link>
     <joint name="caster_rear_joint" type="fixed">

Commit message: Add IMU to robot and integrate with Gazebo plugin
- Modified bumperbot.urdf.xacro to include IMU sensor
- Updated bumperbot_gazebo.xacro to integrate IMU with Gazebo plugin

File: bumperbot_description/urdf/bumperbot.urdf.xacro (robot description, xacro)
@@ -126,3 +126,31 @@
         <origin xyz="-0.04755 0 -0.0275" rpy="0 0 0"/>
     </joint>
+    <link name="imu_link">
+        <inertial>
+            <origin xyz="-0.00552433659106688 0.000168210391520346 0.000514000497342681" rpy="0 0 0"/>
+            <mass value="0.000528415362211671"/>
+            <inertia ixx="1.46176048428261E-08" ixy="1.40015117949421E-10" ixz="-1.99633872937403E-12" iyy="8.59662482954888E-09" iyz="7.52375112767959E-12" izz="2.30279421279312E-08"/>
+        </inertial>
+        <visual>
+            <origin xyz="0 0 0" rpy="0 0 0"/>
+            <geometry>
+                <mesh filename="package://bumperbot_description/meshes/imu_link.STL"/>
+            </geometry>
+            <material name="">
+                <color rgba="0.792156862745098 0.819607843137255 0.933333333333333 1"/>
+            </material>
+        </visual>
+        <collision>
+            <origin xyz="0 0 0" rpy="0 0 0"/>
+            <geometry>
+                <mesh filename="package://bumperbot_description/meshes/imu_link.STL"/>
+            </geometry>
+        </collision>
+    </link>
+    <joint name="imu_joint" type="fixed">
+        <origin xyz="0 0 0.0698986241758014" rpy="0 0 0"/>
+        <parent link="base_link"/>
+        <child link="imu_link"/>
+        <axis xyz="0 0 0"/>
+    </joint>
 </robot>

File: bumperbot_description/urdf/bumperbot_gazebo.xacro (robot description, xacro)
@@ -56,3 +56,52 @@
         </plugin>
     </gazebo>
+    <gazebo reference="imu_link">
+        <sensor name="imu" type="imu">
+            <always_on>true</always_on>
+            <update_rate>100</update_rate>
+            <imu>
+                <angular_velocity>
+                    <x>
+                        <noise type="gaussian">
+                            <mean>0.0</mean>
+                            <stddev>2e-4</stddev>
+                        </noise>
+                    </x>
+                    <y>
+                        <noise type="gaussian">
+                            <mean>0.0</mean>
+                            <stddev>2e-4</stddev>
+                        </noise>
+                    </y>
+                    <z>
+                        <noise type="gaussian">
+                            <mean>0.0</mean>
+                            <stddev>2e-4</stddev>
+                        </noise>
+                    </z>
+                </angular_velocity>
+                <linear_acceleration>
+                    <x>
+                        <noise type="gaussian">
+                            <mean>0.0</mean>
+                            <stddev>1.7e-2</stddev>
+                        </noise>
+                    </x>
+                    <y>
+                        <noise type="gaussian">
+                            <mean>0.0</mean>
+                            <stddev>1.7e-2</stddev>
+                        </noise>
+                    </y>
+                    <z>
+                        <noise type="gaussian">
+                            <mean>0.0</mean>
+                            <stddev>1.7e-2</stddev>
+                        </noise>
+                    </z>
+                </linear_acceleration>
+            </imu>
+            <plugin name="imu" filename="libgazebo_ros_imu_sensor.so"/>
+        </sensor>
+    </gazebo>
 </robot>

Commit message: Add 2D LiDAR (RPLidar A2) to simulation
- Modified bumperbot.urdf.xacro and bumperbot_gazebo.xacro in bumperbot_description package to include the 2D LiDAR sensor.
- Added laser_link.STL mesh file to bumperbot_description package.

File: bumperbot_description/urdf/bumperbot.urdf.xacro (robot description, xacro)
@@ -155,3 +155,28 @@
         <axis xyz="0 0 0"/>
     </joint>
+    <link name="laser_link">
+        <inertial>
+            <origin xyz="-0.011945780406062 -0.000381929217680526 -0.0170649378129477" rpy="0.0 0.0 0.0"/>
+            <mass value="0.073084435549317"/>
+            <inertia ixx="1.96074931730795E-05" ixy="-3.62091076640009E-07" ixz="4.28230084046735E-07"
+                     iyy="2.40983835136327E-05" iyz="1.50180909250652E-08" izz="4.14184164228595E-05"/>
+        </inertial>
+        <visual>
+            <origin xyz="0.0 0.0 0.0" rpy="0.0 0.0 0.0"/>
+            <geometry>
+                <mesh filename="package://bumperbot_description/meshes/laser_link.STL"/>
+            </geometry>
+        </visual>
+        <collision>
+            <origin xyz="0.0 0.0 0.0" rpy="0.0 0.0 0.0"/>
+            <geometry>
+                <mesh filename="package://bumperbot_description/meshes/laser_link.STL"/>
+            </geometry>
+        </collision>
+    </link>
+    <joint name="laser_joint" type="fixed">
+        <parent link="base_link"/>
+        <child link="laser_link"/>
+        <origin xyz="0.0 0.0 0.1208" rpy="0.0 0.0 3.14"/>
+    </joint>
 </robot>

File: bumperbot_description/urdf/bumperbot_gazebo.xacro (robot description, xacro)
@@ -105,3 +105,37 @@
         </sensor>
     </gazebo>
+    <gazebo reference="laser_link">
+        <sensor name="lidar" type="ray">
+            <always_on>true</always_on>
+            <visualize>true</visualize>
+            <update_rate>5</update_rate>
+            <ray>
+                <scan>
+                    <horizontal>
+                        <samples>360</samples>
+                        <resolution>1.0</resolution>
+                        <min_angle>0.0</min_angle>
+                        <max_angle>6.28</max_angle>
+                    </horizontal>
+                </scan>
+                <range>
+                    <min>0.12</min>
+                    <max>12.0</max>
+                    <resolution>0.02</resolution>
+                </range>
+                <noise>
+                    <type>gaussian</type>
+                    <mean>0.0</mean>
+                    <stddev>0.01</stddev>
+                </noise>
+            </ray>
+            <plugin name="scan" filename="libgazebo_ros_ray_sensor.so">
+                <ros>
+                    <remapping>~/out:=scan</remapping>
+                </ros>
+                <output_type>sensor_msgs/LaserScan</output_type>
+                <frame_name>laser_link</frame_name>
+            </plugin>
+        </sensor>
+    </gazebo>
 </robot>

Commit message: Implement dynamic speed control based on zone danger/warning levels and display markers in RViz
- Updated bumperbot.urdf.xacro in bumperbot_description package to reflect changes.
- Modified CMakeLists.txt and package.xml in bumperbot_utils package for new safety stop functionality.
- Enhanced safety_stop.cpp in bumperbot_utils package to include dynamic speed control based on danger and warning zones.
- Added safety_maker.rviz file in bumperbot_description/rviz to visualize danger and warning zones in RViz.

File: bumperbot_description/urdf/bumperbot.urdf.xacro (robot description, xacro)
@@ -136,5 +136,5 @@
             <origin xyz="0 0 0" rpy="0 0 0"/>
             <geometry>
-                <mesh filename="package://bumperbot_description/meshes/imu_link.STL"/>
+                <mesh filename="file://$(find bumperbot_description)/meshes/imu_link.STL"/>
             </geometry>
             <material name="">
@@ -145,5 +145,5 @@
             <origin xyz="0 0 0" rpy="0 0 0"/>
             <geometry>
-                <mesh filename="package://bumperbot_description/meshes/imu_link.STL"/>
+                <mesh filename="file://$(find bumperbot_description)/meshes/imu_link.STL"/>
             </geometry>
         </collision>
@@ -165,5 +165,5 @@
             <origin xyz="0.0 0.0 0.0" rpy="0.0 0.0 0.0"/>
             <geometry>
-                <mesh filename="package://bumperbot_description/meshes/laser_link.STL"/>
+                <mesh filename="file://$(find bumperbot_description)/meshes/laser_link.STL"/>
             </geometry>
         </visual>
@@ -171,5 +171,5 @@
             <origin xyz="0.0 0.0 0.0" rpy="0.0 0.0 0.0"/>
             <geometry>
-                <mesh filename="package://bumperbot_description/meshes/laser_link.STL"/>
+                <mesh filename="file://$(find bumperbot_description)/meshes/laser_link.STL"/>
             </geometry>
         </collision>
